File: KICAD/Reforge_1.kicad_sch (KiCad schematic)
At the start: 91 parts, among them J2 Conn_01x19, J3 Conn_01x02, J4 Conn_01x24, J5 Conn_01x24, J8 Conn_01x19, P1 USB_C_Plug_USB2.0, Q1 SS8050, Q2 SS8050, SW1 SW_Push, SW2 SW_Push, U1 ESP32-WROOM-32E, U2 CP2102N-Axx-xQFN28, U3 ICE40UP5K-SG48ITR, U4 AP2112K-1.2, U5 AP2112K-3.3, U6 SN74LV4T125, U7 SN74LVC1G125DRL, U8 W25Q32JVSS, Y1 SG-210STF

Commit message: Added SCHEMATIC with footprints of our PCB
Parts:
- removed P1: USB_C_Plug_USB2.0, symbol Connector:USB_C_Plug_USB2.0
- removed R24: 5.1K, symbol Device:R
- added J1: USB_B_Micro, Connector_USB:USB_Micro-B_Molex_47346-0001, symbol Connector:USB_B_Micro
- C1, C4, C5: footprint (none) -> Capacitor_SMD:C_0805_2012Metric
- C10, C11, C12, C14, C17, C18, C2, C20, C21, C24, C25, C26, C27, C28, C3, C9: footprint (none) -> Capacitor_SMD:C_0402_1005Metric
- C13, C15, C16, C19, C22, C23, C6, C7, C8: footprint (none) -> Capacitor_SMD:C_0603_1608Metric
- D2, VBUS1: footprint (none) -> LED_SMD:LED_RGB_Wuerth-PLCC4_3.2x2.8mm_150141M173100
- D3, D4, D5, D6: footprint (none) -> Diode_SMD:D_SOD-323
- D7, PWR_LED1: footprint (none) -> LED_SMD:LED_0603_1608Metric
- J2, J8: footprint (none) -> Connector_PinHeader_2.54mm:PinHeader_1x19_P2.54mm_Horizontal
- J3: footprint (none) -> Connector_PinHeader_2.54mm:PinHeader_1x02_P2.54mm_Vertical
- J4, J5: footprint (none) -> Connector_PinHeader_2.54mm:PinHeader_1x24_P2.54mm_Horizontal
- R1, R10, R11, R12, R14, R15, R16, R17, R18, R19, R2, R20, R21, R22, R23, R3, R4, R5, R6, R7, R8, R9: footprint (none) -> Resistor_SMD:R_0402_1005Metric
- R13, SJ19, SJ26, SJ27, SJ28, SJ29: footprint (none) -> Jumper:SolderJumper-2_P1.3mm_Open_Pad1.0x1.5mm
- SJ20, SJ31, SJ34: footprint (none) -> Jumper:SolderJumper-2_P1.3mm_Bridged2Bar_Pad1.0x1.5mm
- SW1, SW2: footprint (none) -> Button_Switch_SMD:SW_SPST_B3U-1000P
- TP1, TP2, TP6: footprint (none) -> TestPoint:TestPoint_Pad_D1.0mm
- U6: footprint (none) -> Package_SO:TSSOP-14_4.4x5mm_P0.65mm
Connections:
- net GND: now also J1.5 (GND), J1.SH (Shield)
- net USB_DN: now also D3.2 (A2), J1.2 (D-); no longer D5.2 (A2)
- net USB_DP: now also D5.2 (A2), J1.3 (D+); no longer D3.2 (A2)
- net VBUS: now also J1.1 (VBUS)
Other:
- moved on the sheet: D3, D4, D5, D6, Q1, Q2, R10, R7, R8, R9
